File: pcb/rev.A/picogus104.kicad_pcb (KiCad board)
At the start: 4 copper layers, 56 x 87.8 mm, 112 parts, among them J1 USB_C_Receptacle_USB2.0_16P, J10 Conn_01x02_Pin, J11 PC104, J12 PC104_16, J2 DEBUG, J3 IRQDMA_JP, J4 UART_TX, J7 3.5mm TRS, J9 3.5mm TRS, Q1 AO3401A, SW1 SW_Push, U1 SN74CB3T3257, U10 PCM5100, U11 W25Q128JVS, U12 RP2040, U13 M62429L, U14 SAM2695, U2 SN74CB3T3257, U3 74AHC14, U4 74LVC00, U5 74LVC00, U6 74LVC2G06DB, U7 SN74CB3T3245, U8 APS6404L-3SQR-SN, U9 AMS1117-3.3_SOT223, Y1 ABLS-12.000MHZ-B4-T, Y2 12 MHz

Commit message: wip pcb reb.A - almost done
Parts:
- removed D2: D_Schottky, Diode_SMD:D_SOD-123
- removed Q1: AO3401A, Package_TO_SOT_SMD:SOT-23
- added J5: Conn_01x02_Pin, Connector_PinHeader_2.54mm:PinHeader_1x02_P2.54mm_Vertical, F.Cu at (153.3, 72.6)
- added R21: 5.1k, Resistor_SMD:R_0603_1608Metric_Pad0.98x0.95mm_HandSolder, F.Cu at (150.1, 70.6)
- R17: value 15K -> 5.1k
- R19, R20: footprint Resistor_SMD:R_0805_2012Metric_Pad1.20x1.40mm_HandSolder -> Resistor_SMD:R_0603_1608Metric_Pad0.98x0.95mm_HandSolder
- moved C4 21.2 mm to (156.4, 96.7), turned to 90 degrees
- moved U7 18.7 mm to (152.1, 94.7)
- moved U5 18.6 mm to (145.8, 94.7)
- moved C8 18.6 mm to (146.8, 99.4)
- moved R5 11.2 mm to (146.8, 90.0)
- moved C9 11.2 mm to (153.9, 119.6)
- moved R1 11.1 mm to (143.4, 119.6)
- moved C6 11.1 mm to (146.8, 119.6)
- moved U2 11.1 mm to (152.8, 114.8)
- moved U3 11.0 mm to (145.8, 114.8)
- moved C7 10.1 mm to (146.8, 109.3)
- moved U1 10.0 mm to (152.8, 104.6)
- moved U4 9.96 mm to (145.7, 104.6)
- moved C41 9.80 mm to (126.2, 74.4)
- moved C42 9.80 mm to (131.1, 74.4)
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Connections:
- C12 pad 1: /VSYS -> +5V
- F1 pad 2: Net-(D2-A) -> Net-(J5-Pin_2)
- J9 pad RN: unconnected-(J9-PadRN) -> Net-(J9-PadR)
- J9 pad TN: unconnected-(J9-PadTN) -> Net-(J9-PadT)
- R17 pad 1: Net-(D2-A) -> Net-(J1-CC2)
- R17 pad 2: GND -> Net-(F1-Pad1)
- U9 pad 3: /VSYS -> +5V
Routing:
- net GND: track 0.00 -> 179.4 mm, vias 0 -> 126
- net +3V3: track 0.00 -> 124.2 mm, vias 0 -> 63
- net UART_TX: track 0.00 -> 85.8 mm, vias 0 -> 4
- net /USB_D+: track 0.00 -> 77.2 mm, vias 0 -> 4
- net /USB_D-: track 0.00 -> 75.6 mm, vias 0 -> 2
- net Net-(U13-2ch_IN): track 0.00 -> 71.1 mm
- net RUN: track 0.00 -> 69.1 mm, vias 0 -> 4
- net IRQ3: track 0.00 -> 68.6 mm
- net IRQ4: track 0.00 -> 63.9 mm
- net /RP2040/~{USB_BOOT}: track 0.00 -> 62.5 mm
- net IRQ5: track 0.00 -> 59.2 mm
- net /RP2040/GPIO23: track 0.00 -> 58.8 mm, vias 0 -> 2
- net Net-(U13-1ch_IN): track 0.00 -> 58.0 mm
- net ~{BUSOE}: track 0.00 -> 53.5 mm, vias 0 -> 5
- net ADS: track 0.00 -> 53.0 mm, vias 0 -> 5
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Other:
- board text added: "2"
- board text added: "USB POWER"

Commit message: pcb rev.A - final version
Parts:
- added J6: Conn_01x04_Pin, Connector_PinHeader_2.54mm:PinHeader_1x04_P2.54mm_Vertical, F.Cu at (121.5, 58.7)
- added J8: Conn_01x04_Pin, Connector_PinHeader_2.54mm:PinHeader_1x04_P2.54mm_Vertical, F.Cu at (136.6, 58.7)
- J7, J9: footprint my:PJ-307 -> my:PJ-322
- Y2: value 12 MHz -> ABLS-12.000MHZ-B4-T
- moved J9 2.57 mm to (127.5, 62.0)
- moved J7 2.48 mm to (142.4, 62.0)
- moved FB1 1.01 mm to (141.4, 72.6)
- moved FB2 1.01 mm to (143.7, 72.6)
- moved R2 1.01 mm to (141.4, 76.6)
- moved R3 1.01 mm to (143.7, 76.6)
- moved R6 0.60 mm to (131.1, 70.4)
- moved R7 0.60 mm to (126.2, 70.4)
- moved R8 0.60 mm to (136.0, 70.4)
- moved R9 0.60 mm to (121.3, 70.4)
- moved C41 0.30 mm to (126.2, 74.7)
- moved C42 0.30 mm to (131.1, 74.7)
- moved C43 0.30 mm to (121.3, 74.7)
- moved C44 0.30 mm to (136.0, 74.7)
Connections:
- FB1 pad 2: Net-(FB1-Pad2) -> Net-(J8-Pin_1)
- FB2 pad 2: Net-(FB2-Pad2) -> Net-(J8-Pin_4)
- J7 pad T: Net-(FB1-Pad2) -> Net-(J8-Pin_1)
- J9 pad T: Net-(J9-PadT) -> Net-(J6-Pin_1)
- R6 pad 2: Net-(J9-PadR) -> Net-(J6-Pin_4)
- R7 pad 2: Net-(J9-PadT) -> Net-(J6-Pin_1)
- R8 pad 1: Net-(J9-PadR) -> Net-(J6-Pin_4)
- R9 pad 1: Net-(J9-PadT) -> Net-(J6-Pin_1)
Routing:
- net Net-(J6-Pin_1): track 0.00 -> 25.3 mm
- net Net-(J8-Pin_1): track 0.00 -> 21.9 mm
- net Net-(J6-Pin_4): track 0.00 -> 16.4 mm
- net Net-(J9-PadT): track 13.9 -> 0.00 mm
- net Net-(J9-PadR): track 13.6 -> 0.00 mm
- net Net-(J8-Pin_4): track 0.00 -> 12.4 mm
- net Net-(FB1-Pad2): track 9.18 -> 0.00 mm
- net Net-(FB2-Pad2): track 8.06 -> 0.00 mm
- net GND: track 179.4 -> 182.8 mm, vias 126 -> 127
- net AGND: track 63.4 -> 65.9 mm
- net PGAUDIO_L: track 14.2 -> 13.6 mm
Other:
- board text added: "G"
- board text added: "L"
- board text added: "R"
- board text added: "Sink"
- board text added: "Source"

Commit message: bom fixes
Parts:
- C12, C13, C47, C49: value 10u -> 10uF
- C18: footprint Capacitor_SMD:C_0805_2012Metric -> Capacitor_SMD:C_0805_2012Metric_Pad1.18x1.45mm_HandSolder
- C50, C51: value 30p -> 30pF
- Y1, Y2: value ABLS-12.000MHZ-B4-T -> 12MHz
