File: pcb/rev.A/picogus104.kicad_sch (KiCad schematic)
At the start: 91 parts, among them J1 USB_C_Receptacle_USB2.0_16P, J10 Conn_01x02_Pin, J11 PC104, J12 PC104_16, J2 DEBUG, J3 IRQDMA_JP, J4 UART_TX, J7 3.5mm TRS, J9 3.5mm TRS, Q1 AO3401A, SW1 SW_Push, U1 SN74CB3T3257, U10 PCM5100, U13 M62429L, U14 SAM2695, U2 SN74CB3T3257, U3 74AHC14, U4 74LVC00, U5 74LVC00, U6 74LVC2G06DB, U7 SN74CB3T3245, U8 APS6404L-3SQR-SN, Y2 12 MHz

Commit message: wip pcb reb.A - almost done
Parts:
- removed D2: D_Schottky, Diode_SMD:D_SOD-123, symbol Device:D_Schottky
- removed Q1: AO3401A, Package_TO_SOT_SMD:SOT-23, symbol Transistor_FET:AO3401A
- added J5: Conn_01x02_Pin, Connector_PinHeader_2.54mm:PinHeader_1x02_P2.54mm_Vertical, symbol Connector:Conn_01x02_Pin
- added R21: 5.1k, Resistor_SMD:R_0603_1608Metric_Pad0.98x0.95mm_HandSolder, symbol Device:R
- R17: value 15K -> 5.1k; ValueSilk (none) -> ${VALUE}; now not fitted
- R19, R20: footprint Resistor_SMD:R_0805_2012Metric_Pad1.20x1.40mm_HandSolder -> Resistor_SMD:R_0603_1608Metric_Pad0.98x0.95mm_HandSolder; now not fitted
Connections:
- net VSYS is gone; now on net +5V: C?.1, U?.3 (VI)
- net +5V: now also J5.1 (Pin_1)
- net GND: no longer R17.2
- net at J9.T, R7.2, R9.1: now also J9.TN
- net at J1.A5 (CC1), R19.2: now also R21.1
- net at J9.R, R6.2, R8.1: now also J9.RN
- net at J1.B5 (CC2), R20.2: now also R17.1
- net at F1.2: now also J5.2 (Pin_2); no longer R17.1
- net at F1.1, J1.A4 (VBUS), J1.A9 (VBUS)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: now also R17.2, R21.2
- no-connect marks 78 -> 76
Other:
- moved on the sheet: F1, J1

Commit message: pcb rev.A - final version
Parts:
- added J6, J8: Conn_01x04_Pin, Connector_PinHeader_2.54mm:PinHeader_1x04_P2.54mm_Vertical, symbol Connector:Conn_01x04_Pin
- J7, J9: footprint my:PJ-307 -> my:PJ-322; symbol Connector_Audio:AudioJack3_SwitchTR -> Connector_Audio:AudioJack4
- Y2: value 12 MHz -> ABLS-12.000MHZ-B4-T
Connections:
- net AGND: now also J9.R2, J6.2 (Pin_2), J6.3 (Pin_3)
- net GND: now also J7.R2, J8.2 (Pin_2), J8.3 (Pin_3)
- net at J9.T, R7.2, R9.1: now also J6.1 (Pin_1); no longer J9.TN
- net at FB1.2, J7.T: now also J8.1 (Pin_1); no longer J7.TN
- net at R6.2, R8.1: now also J9.R1, J6.4 (Pin_4); no longer J9.R, J9.RN
- new net: FB2.2, J7.R1, J8.4 (Pin_4)
Other:
- title: PicoGUS v1.1 -> PicoGUS/104

Commit message: bom fixes
Parts:
- C18: footprint Capacitor_SMD:C_0805_2012Metric -> Capacitor_SMD:C_0805_2012Metric_Pad1.18x1.45mm_HandSolder
- C47, C49, C? (x2): value 10u -> 10uF
- C50, C51: value 30p -> 30pF
- R17, R19, R20, R21: now left out of the parts list
Changed lines of the file:
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@@
 			)
 		)
-		(property "Value" "30p"
+		(property "Value" "30pF"
 			(at 288.29 87.63 0)
 			(effects
@@
 			)
 		)
-		(property "Footprint" "Capacitor_SMD:C_0805_2012Metric"
+		(property "Footprint" "Capacitor_SMD:C_0805_2012Metric_Pad1.18x1.45mm_HandSolder"
 			(at 356.87 135.89 0)
 			(effects
@@
 		(unit 1)
 		(exclude_from_sim no)
-		(in_bom yes)
+		(in_bom no)
 		(on_board yes)
 		(dnp yes)
@@
 			)
 		)
-		(property "Value" "10u"
+		(property "Value" "10uF"
 			(at 273.05 57.15 0)
 			(effects
@@
 			)
 		)
-		(property "Value" "30p"
+		(property "Value" "30pF"
 			(at 278.13 87.63 0)
 			(effects
@@
 		(unit 1)
 		(exclude_from_sim no)
-		(in_bom yes)
+		(in_bom no)
 		(on_board yes)
 		(dnp yes)
@@
 		(unit 1)
 		(exclude_from_sim no)
-		(in_bom yes)
+		(in_bom no)
 		(on_board yes)
 		(dnp yes)
@@
 			)
 		)
-		(property "Value" "10u"
+		(property "Value" "10uF"
 			(at 271.78 87.63 0)
 			(effects
@@
 		(unit 1)
 		(exclude_from_sim no)
-		(in_bom yes)
+		(in_bom no)
 		(on_board yes)
 		(dnp yes)
@@
 			)
 		)
-		(property "Value" "10u"
+		(property "Value" "10uF"
 			(at 390.271 222.123 0)
 			(effects
@@
 			)
 		)
-		(property "Value" "10u"
+		(property "Value" "10uF"
 			(at 363.601 222.123 0)
 			(effects
